File: Projetos Eagle/POTENCIOMETRO.sch (EAGLE design)
At the start: 9 parts, among them IC1 TL494BD, J1 CONECTOR_MACHO, J2 CONECTOR_FEMEA

Commit message: correção de pads, adição de label para versionamento, adição de resistor R4 para ajuste de sensibilidade e correção de entradas do POT
Parts:
- added R4: 4K7, rcl:R-EU_R0805W
- renumbered IC1 to U1
Connections:
- removed net N$1: U1.+I1, U1.+I2
- net GND: now also POT.CCW, U1.+I1, U1.+I2; no longer POT.CW
- net POT_SIGNAL: now also R4.1
- net SIGNAL_IN: now also POT.CW, R4.2; no longer POT.CCW

Commit message: adição de filtro no SIGNAL_OUT para correção do Duty Clycle
Parts:
- added C3: 100nF, rcl:C-EUC0805
- added R5: 1k, rcl:R-EU_R0805W
Connections:
- new net PWM: R3.2, R5.1, U1.C1
- net GND: now also C3.1
- net SIGNAL_OUT: now also C3.2, R5.2; no longer R3.2, U1.C1
Changed lines of the file:
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@@
 <setting verticaltext="up"/>
 </settings>
-<grid distance="0.01" unitdist="mm" unit="mm" style="lines" multiple="1" display="no" altdistance="0.1" altunitdist="mm" altunit="mm"/>
+<grid distance="0.1" unitdist="inch" unit="inch" style="lines" multiple="1" display="no" altdistance="0.01" altunitdist="inch" altunit="inch"/>
 <layers>
 <layer number="1" name="Top" color="4" fill="1" visible="no" active="no"/>
@@
 <schematic_group name="PWM_SIGNAL"/>
 <schematic_group name="POT_SINGAL"/>
+<schematic_group name="FILTER"/>
 </groups>
 <parts>
@@
 <part name="GND7" library="supply1" library_urn="urn:adsk.eagle:library:371" deviceset="GND" device=""/>
 <part name="R4" library="rcl" library_urn="urn:adsk.eagle:library:334" deviceset="R-EU_" device="R0805W" package3d_urn="urn:adsk.eagle:package:23537/2" value="4K7"/>
+<part name="R5" library="rcl" library_urn="urn:adsk.eagle:library:334" deviceset="R-EU_" device="R0805W" package3d_urn="urn:adsk.eagle:package:23537/2" value="1k"/>
+<part name="C3" library="rcl" library_urn="urn:adsk.eagle:library:334" deviceset="C-EU" device="C0805" package3d_urn="urn:adsk.eagle:package:23617/2" value="100nF"/>
+<part name="GND8" library="supply1" library_urn="urn:adsk.eagle:library:371" deviceset="GND" device=""/>
 </parts>
 <sheets>
@@
 <attribute name="NAME" x="51.28100625" y="70.853259375" size="1.778" layer="95" rot="R90"/>
 <attribute name="VALUE" x="54.040890625" y="73.76108125" size="1.778" layer="96" rot="R270"/>
+</instance>
+<instance part="R5" gate="G$1" x="18.514575" y="-23.477365625" smashed="yes" grouprefs="FILTER">
+<attribute name="NAME" x="19.908559375" y="-24.873271875" size="1.778" layer="95" rot="R180"/>
+<attribute name="VALUE" x="17.0007375" y="-22.1133875" size="1.778" layer="96"/>
+</instance>
+<instance part="C3" gate="G$1" x="25.16181875" y="-30.394278125" smashed="yes" rot="R180" grouprefs="FILTER">
+<attribute name="NAME" x="20.84281875" y="-27.598278125" size="1.778" layer="95" rot="R270"/>
+<attribute name="VALUE" x="27.36281875" y="-25.898278125" size="1.778" layer="96" rot="R270"/>
+</instance>
+<instance part="GND8" gate="1" x="25.01671875" y="-38.343278125" smashed="yes" grouprefs="FILTER">
+<attribute name="VALUE" x="22.47671875" y="-41.083278125" size="1.778" layer="96"/>
 </instance>
 </instances>
@@
 <junction x="23.66" y="38.52"/>
 </segment>
+<segment>
+<pinref part="GND8" gate="1" pin="GND"/>
+<pinref part="C3" gate="G$1" pin="1"/>
+<wire x1="25.01671875" y1="-35.803278125" x2="25.01671875" y2="-32.934278125" width="0.1524" layer="91" grouprefs="FILTER"/>
+<wire x1="25.01671875" y1="-32.934278125" x2="25.16181875" y2="-32.934278125" width="0.1524" layer="91" grouprefs="FILTER"/>
+</segment>
 </net>
 <net name="SIGNAL_OUT" class="0">
@@
 </segment>
 <segment>
-<pinref part="U1" gate="G$1" pin="C1"/>
-<wire x1="54.14" y1="23.28" x2="94.24" y2="23.28" width="0.1524" layer="91" grouprefs="PWM_SIGNAL"/>
-<label x="94.14" y="23.38" size="1.778" layer="95" xref="yes" grouprefs="PWM_SIGNAL"/>
-<pinref part="R3" gate="G$1" pin="2"/>
-<wire x1="54.14" y1="23.28" x2="85.603334375" y2="23.28" width="0.1524" layer="91"/>
-<wire x1="85.603334375" y1="23.28" x2="85.603334375" y2="27.67533125" width="0.1524" layer="91"/>
-<junction x="54.14" y="23.28"/>
+<pinref part="R5" gate="G$1" pin="2"/>
+<pinref part="C3" gate="G$1" pin="2"/>
+<wire x1="23.594575" y1="-23.477365625" x2="25.16181875" y2="-23.477365625" width="0.1524" layer="91" grouprefs="FILTER"/>
+<wire x1="25.16181875" y1="-23.477365625" x2="25.16181875" y2="-25.314278125" width="0.1524" layer="91" grouprefs="FILTER"/>
+<wire x1="23.594575" y1="-23.477365625" x2="38.32351875" y2="-23.477365625" width="0.1524" layer="91" grouprefs="FILTER"/>
+<wire x1="38.32351875" y1="-23.477365625" x2="38.32351875" y2="-23.5483375" width="0.1524" layer="91" grouprefs="FILTER"/>
+<junction x="23.594575" y="-23.477365625" grouprefs="FILTER"/>
+<label x="38.460678125" y="-23.309578125" size="1.27" layer="95" xref="yes" grouprefs="FILTER"/>
 </segment>
 </net>
@@
 </segment>
 </net>
+<net name="PWM" class="0">
+<segment>
+<pinref part="R5" gate="G$1" pin="1"/>
+<wire x1="13.434575" y1="-23.477365625" x2="8.488678125" y2="-23.477365625" width="0.1524" layer="91" grouprefs="FILTER"/>
+<wire x1="8.488678125" y1="-23.477365625" x2="8.488678125" y2="-23.571196875" width="0.1524" layer="91" grouprefs="FILTER"/>
+<label x="8.417559375" y="-23.441659375" size="1.27" layer="95" rot="R180" xref="yes" grouprefs="FILTER"/>
+</segment>
+<segment>
+<pinref part="U1" gate="G$1" pin="C1"/>
+<wire x1="54.14" y1="23.28" x2="94.24" y2="23.28" width="0.1524" layer="91" grouprefs="PWM_SIGNAL"/>
+<label x="94.14" y="23.38" size="1.778" layer="95" xref="yes" grouprefs="PWM_SIGNAL"/>
+<pinref part="R3" gate="G$1" pin="2"/>
+<wire x1="54.14" y1="23.28" x2="85.603334375" y2="23.28" width="0.1524" layer="91"/>
+<wire x1="85.603334375" y1="23.28" x2="85.603334375" y2="27.67533125" width="0.1524" layer="91"/>
+<junction x="54.14" y="23.28"/>
+</segment>
+</net>
