File: Projetos Eagle/POTENCIOMETRO.brd (EAGLE design)
At the start: 47.8 x 21.5 mm, 11 parts, among them J1 CONECTOR_MACHO, J2 CONECTOR_FEMEA, U1 TL494BD

Commit message: adição de filtro no SIGNAL_OUT para correção do Duty Clycle
Parts:
- added C3: 100nF, rcl:C0805
- added R5: 1k, rcl:R0805W
- added U$2: (no value), Eletroblocks Lib:VERSAOATT
Connections:
- new net PWM: R3.2, R5.1, U1.8
- net GND: now also C3.1
- net SIGNAL_OUT: now also C3.2, R5.2; no longer R3.2, U1.8
Routing:
- net PWM: track 0.00 -> 22.7 mm, vias 0 -> 2
- net SIGNAL_OUT: track 18.1 -> 40.8 mm
- net SIGNAL_IN: track 30.5 -> 33.6 mm
Other:
- board text removed: "V1.0.1"
Changed lines of the file:
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@@
 <vertex x="4.5651375" y="10.4536625"/>
 </polygon>
-<text x="-0.4" y="21.4" size="0.6096" layer="22" font="fixed" rot="MR270">V1.0.1</text>
 </plain>
 <attributes>
@@
 <attribute name="VALUE" x="16.365" y="8.54" size="1.27" layer="28" rot="MR180"/>
 </element>
+<element name="R5" library="rcl" library_urn="urn:adsk.eagle:library:334" package="R0805W" package3d_urn="urn:adsk.eagle:package:23537/2" value="1k" x="4" y="12.5" smashed="yes" rot="MR0">
+<attribute name="NAME" x="1.93" y="13.435" size="0.6096" layer="26" font="fixed" rot="MR270"/>
+<attribute name="POPULARITY" value="3" x="4" y="12.5" size="1.778" layer="28" rot="MR0" display="off"/>
+<attribute name="SPICEPREFIX" value="R" x="4" y="12.5" size="1.778" layer="28" rot="MR0" display="off"/>
+<attribute name="VALUE" x="4.635" y="9.96" size="1.27" layer="28" rot="MR0"/>
+</element>
+<element name="C3" library="rcl" library_urn="urn:adsk.eagle:library:334" package="C0805" package3d_urn="urn:adsk.eagle:package:23617/2" value="100nF" x="4" y="10" smashed="yes" rot="MR0">
+<attribute name="NAME" x="1.93" y="11.07" size="0.6096" layer="26" font="fixed" rot="MR270"/>
+<attribute name="POPULARITY" value="88" x="4" y="10" size="1.778" layer="28" rot="MR0" display="off"/>
+<attribute name="SPICEPREFIX" value="C" x="4" y="10" size="1.778" layer="28" rot="MR0" display="off"/>
+<attribute name="VALUE" x="5.27" y="7.46" size="1.27" layer="28" rot="MR0"/>
+</element>
+<element name="U$2" library="Eletroblocks Lib" package="VERSAOATT" value="" x="-2.7" y="21.3" smashed="yes" rot="R90"/>
 </elements>
 <signals>
@@
 <contactref element="U1" pad="16"/>
 <wire x1="23.9266" y1="6.455" x2="30.0734" y2="6.455" width="0.6096" layer="16"/>
+<contactref element="C3" pad="1"/>
 </signal>
 <signal name="VCC">
@@
 </polygon>
 <wire x1="27.95" y1="1.8" x2="30" y2="1.8" width="0.6096" layer="16"/>
-<wire x1="33.6" y1="5.4" x2="33.6" y2="7.1" width="0.6096" layer="16"/>
-<wire x1="33.6" y1="7.1" x2="34.71" y2="8.21" width="0.6096" layer="16"/>
-<wire x1="34.71" y1="8.21" x2="36.3" y2="8.21" width="0.6096" layer="16"/>
+<wire x1="33.6" y1="5.4" x2="33.6" y2="7.2" width="0.6096" layer="16"/>
+<wire x1="33.6" y1="7.2" x2="34.61" y2="8.21" width="0.6096" layer="16"/>
+<wire x1="34.61" y1="8.21" x2="36.3" y2="8.21" width="0.6096" layer="16"/>
 <wire x1="30" y1="1.8" x2="33.6" y2="5.4" width="0.6096" layer="16"/>
 <wire x1="36.3" y1="8.21" x2="31.99" y2="8.21" width="0.6096" layer="1"/>
@@
 <wire x1="29.8" y1="17.9" x2="29.4" y2="17.5" width="0.6096" layer="16"/>
 <wire x1="30.0734" y1="11.535" x2="31.665" y2="11.535" width="0.6096" layer="16"/>
-<wire x1="32.3" y1="10.9" x2="32.3" y2="9.449475" width="0.6096" layer="16"/>
-<wire x1="33.539475" y1="8.21" x2="34.71" y2="8.21" width="0.6096" layer="16"/>
+<wire x1="32.3" y1="10.9" x2="32.3" y2="9.949475" width="0.6096" layer="16"/>
+<wire x1="34.039475" y1="8.21" x2="34.61" y2="8.21" width="0.6096" layer="16"/>
 <wire x1="31.665" y1="11.535" x2="32.3" y2="10.9" width="0.6096" layer="16"/>
-<wire x1="32.3" y1="9.449475" x2="33.539475" y2="8.21" width="0.6096" layer="16"/>
+<wire x1="32.3" y1="9.949475" x2="34.039475" y2="8.21" width="0.6096" layer="16"/>
 </signal>
 <signal name="SIGNAL_IN">
@@
 <contactref element="R4" pad="2"/>
 <wire x1="12.81678125" y1="1.592" x2="12.80878125" y2="1.6" width="0.6096" layer="16"/>
-<wire x1="12.80878125" y1="1.6" x2="9.9" y2="1.6" width="0.6096" layer="16"/>
 <wire x1="18.4" y1="3" x2="16.992" y2="1.592" width="0.6096" layer="16"/>
-<wire x1="16.992" y1="1.592" x2="12.81678125" y2="1.592" width="0.6096" layer="16"/>
-<wire x1="9.9" y1="1.6" x2="0.75" y2="10.75" width="0.6096" layer="16"/>
-<wire x1="-4.5" y1="10.75" x2="0.75" y2="10.75" width="0.6096" layer="16"/>
+<wire x1="16.992" y1="1.592" x2="13.8" y2="1.592" width="0.6096" layer="16"/>
+<wire x1="13.8" y1="1.592" x2="12.81678125" y2="1.592" width="0.6096" layer="16"/>
 <wire x1="18.4" y1="3" x2="18.4" y2="5.7475" width="0.6096" layer="16"/>
 <wire x1="18.4" y1="5.7475" x2="18.0525" y2="6" width="0.6096" layer="16"/>
+<wire x1="-4.5" y1="10.75" x2="-0.45" y2="10.75" width="0.6096" layer="16"/>
+<wire x1="2.5" y1="7.8" x2="2.5" y2="2.5" width="0.6096" layer="16"/>
+<wire x1="2.5" y1="2.5" x2="3.408" y2="1.592" width="0.6096" layer="16"/>
+<wire x1="3.408" y1="1.592" x2="12.81678125" y2="1.592" width="0.6096" layer="16"/>
+<wire x1="-0.45" y1="10.75" x2="2.5" y2="7.8" width="0.6096" layer="16"/>
 </signal>
 <signal name="SIGNAL_OUT">
 <contactref element="J2" pad="2"/>
-<contactref element="U1" pad="8"/>
-<wire x1="24.445" y1="18.508840625" x2="23.962159375" y2="18.026" width="0.6096" layer="16"/>
-<contactref element="R3" pad="2"/>
-<wire x1="23.9266" y1="15.345" x2="23.9266" y2="17.6266" width="0.6096" layer="16"/>
-<wire x1="23.9266" y1="17.6266" x2="24.2" y2="17.9" width="0.6096" layer="16"/>
-<wire x1="36.3" y1="10.75" x2="29.1994" y2="10.75" width="0.6096" layer="1"/>
-<wire x1="26.2698" y1="14.4796" x2="26.2698" y2="13.6796" width="0.6096" layer="1"/>
-<wire x1="29.1994" y1="10.75" x2="26.2698" y2="13.6796" width="0.6096" layer="1"/>
-<via x="26.2698" y="14.4796" extent="1-16" drill="0.3"/>
-<wire x1="23.9266" y1="15.345" x2="25.3266" y2="15.345" width="0.6096" layer="16"/>
-<wire x1="25.592" y1="15.0796" x2="25.3266" y2="15.345" width="0.6096" layer="16"/>
-<wire x1="26.2698" y1="14.4796" x2="25.6698" y2="15.0796" width="0.6096" layer="16"/>
-<wire x1="25.6698" y1="15.0796" x2="25.592" y2="15.0796" width="0.6096" layer="16"/>
-<wire x1="24.2" y1="17.9" x2="23.962159375" y2="18.026" width="0" layer="19" extent="16-16"/>
+<contactref element="R5" pad="2"/>
+<contactref element="C3" pad="2"/>
+<wire x1="2.9475" y1="12.5" x2="2.9475" y2="10.1025" width="0.6096" layer="16"/>
+<wire x1="2.9475" y1="10.1025" x2="3.05" y2="10" width="0.6096" layer="16"/>
+<via x="13.5" y="7" extent="1-16" drill="0.3"/>
+<wire x1="13.5" y1="7" x2="27.5" y2="7" width="0.6096" layer="1"/>
+<wire x1="31.3" y1="10.8" x2="27.5" y2="7" width="0.6096" layer="1"/>
+<wire x1="36.3" y1="10.75" x2="31.35" y2="10.75" width="0.6096" layer="1"/>
+<wire x1="3.05" y1="10" x2="3.05" y2="8.75" width="0.6096" layer="16"/>
+<wire x1="11.7" y1="5.2" x2="13.5" y2="7" width="0.6096" layer="16"/>
+<wire x1="3.05" y1="8.75" x2="6.6" y2="5.2" width="0.6096" layer="16"/>
+<wire x1="6.6" y1="5.2" x2="11.7" y2="5.2" width="0.6096" layer="16"/>
+<wire x1="31.3" y1="10.8" x2="31.35" y2="10.75" width="0" layer="19" extent="1-1"/>
 </signal>
 <signal name="VREF">
@@
 <wire x1="18.6" y1="13.2756" x2="22.62428125" y2="13.2756" width="0.6096" layer="1"/>
 </signal>
+<signal name="PWM">
+<contactref element="R5" pad="1"/>
+<contactref element="U1" pad="8"/>
+<contactref element="R3" pad="2"/>
+<wire x1="23.9266" y1="17.6266" x2="23.9266" y2="15.345" width="0.6096" layer="16"/>
+<wire x1="23.9266" y1="17.6266" x2="24.2" y2="17.9" width="0.6096" layer="16"/>
+<wire x1="23.9266" y1="15.345" x2="21.83488125" y2="15.345" width="0.6096" layer="16"/>
+<wire x1="21.83488125" y1="15.345" x2="21.817440625" y2="15.362440625" width="0.6096" layer="16"/>
+<via x="21.817440625" y="15.362440625" extent="1-16" drill="0.3"/>
+<wire x1="21.817440625" y1="15.362440625" x2="20.655" y2="14.2" width="0.6096" layer="1"/>
+<wire x1="13" y1="14.2" x2="12" y2="13.2" width="0.6096" layer="1"/>
+<via x="12" y="13.2" extent="1-16" drill="0.3"/>
+<wire x1="12" y1="13.2" x2="5.7525" y2="13.2" width="0.6096" layer="16"/>
+<wire x1="5.7525" y1="13.2" x2="5.0525" y2="12.5" width="0.6096" layer="16"/>
+<wire x1="20.655" y1="14.2" x2="13" y2="14.2" width="0.6096" layer="1"/>
+</signal>
 </signals>

Commit message: correção de label
Parts:
- removed U$2: (no value), Eletroblocks Lib:VERSAOATT
Other:
- board text added: "V1.1.0"
Changed lines of the file:
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@@
 <vertex x="4.5651375" y="10.4536625"/>
 </polygon>
+<text x="-0.5" y="21.3" size="0.6096" layer="22" font="fixed" rot="MR270">V1.1.0</text>
 </plain>
 <attributes>
@@
 <attribute name="VALUE" x="5.27" y="7.46" size="1.27" layer="28" rot="MR0"/>
 </element>
-<element name="U$2" library="Eletroblocks Lib" package="VERSAOATT" value="" x="-2.7" y="21.3" smashed="yes" rot="R90"/>
 </elements>
 <signals>
